File: 4x4-key-pcb/4x4-key-pcb.kicad_pcb (KiCad board)
At the start: 2 copper layers, 90 x 90 mm, 61 parts, among them J2 Conn_01x05_Pin, SW1 SW_Push, U1 TPS62162DSG, U2 STM32G0B1KBTx, U3 SN65HVD230

Commit message: routed 4x4 pad
Connections:
- U2 pad 28: unconnected-(U2-PB4-Pad28) -> R2
- U2 pad 29: unconnected-(U2-PB5-Pad29) -> R3
- U2 pad 30: unconnected-(U2-PB6-Pad30) -> C2
- U2 pad 31: unconnected-(U2-PB7-Pad31) -> C3
Routing:
- net GND: track 218.1 -> 469.2 mm, vias 0 -> 5
- net CAN_L: track 166.5 -> 362.8 mm, vias 0 -> 1
- net CAN_H: track 194.5 -> 381.9 mm, vias 0 -> 1
- net +5V: track 241.9 -> 379.8 mm, vias 0 -> 3
- net R0: track 0.00 -> 93.5 mm, vias 0 -> 3
- net C3: track 0.00 -> 90.5 mm, vias 0 -> 2
- net R3: track 0.00 -> 89.0 mm
- net C2: track 0.00 -> 79.9 mm
- net C0: track 0.00 -> 78.3 mm, vias 0 -> 2
- net R1: track 0.00 -> 73.7 mm, vias 0 -> 1
- net +3.3V: track 0.00 -> 64.2 mm
- net C1: track 0.00 -> 63.8 mm, vias 0 -> 4
- net R2: track 0.00 -> 62.5 mm
- net PF2: track 0.00 -> 37.1 mm, vias 0 -> 1
- net SWCLK: track 0.00 -> 17.6 mm, vias 0 -> 1
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Other:
- outline, holes or cut-outs redrawn
